File: Hardware/PCB/KiCAD_files/Wazo.kicad_pcb (KiCad board)
At the start: 2 copper layers, 60 x 60 mm, 78 parts, among them IC1 BQ24250RGER, IC2 MAX20402AFLB_VY+T, IC3 MAX98357AETE+T, J1 USB_C_Receptacle_USB2.0, J2 B2B-PH-SM4-TB(LF)(SN), J3 B2B-PH-SM4-TB(LF)(SN), J4 Conn_01x08, SW1 SLW-66527511-SMT-TR, SW2 SLW-66527511-SMT-TR, U1 ESP32-S3-WROOM-1

Commit message: grantmeplease
Parts:
- removed the G*** at (175.8, 77.4)
